Commit message: config: add 2f-140 gripper.
config: add 2f-140 gripper urdf, srdf and gripper controller

File: ur_moveit_config/srdf/ur_macro.srdf.xacro (robot description, xacro)
@@ -11,9 +11,21 @@
     <!--CHAINS - When a chain is specified, all the links along the chain (including endpoints) are included in the group. Additionally, all the joints that are parents to included links are also included. This means that joints along the chain and the parent joint of the base link are included in the group-->
     <!--SUBGROUPS - Groups can also be formed by referencing to already defined group names-->
-    <group name="${prefix}${name}_manipulator">
-      <chain base_link="${prefix}base_link" tip_link="${prefix}tool0" />
+    <group name="ur_manipulator">
+      <chain base_link="${prefix}base_link" tip_link="${prefix}ee_link" />
+    </group>
+    <group name="${prefix}${name}_gripper">
+      <joint name="finger_joint"/>
+      <joint name="left_inner_knuckle_joint" />
+      <joint name="left_inner_finger_joint" />
+      <joint name="left_outer_finger_joint" />
+      <joint name="right_inner_knuckle_joint" />
+      <joint name="right_outer_knuckle_joint" />
+      <joint name="right_inner_finger_joint" />
+      <joint name="right_outer_finger_joint" />
+      <joint name="left_inner_finger_pad_joint" />
+      <joint name="right_inner_finger_pad_joint" />
     </group>
     <!--GROUP STATES - Purpose - Define a named state for a particular group, in terms of joint values. This is useful to define states like 'folded arms'-->
-    <group_state name="${prefix}home" group="${prefix}${name}_manipulator">
+    <group_state name="${prefix}home" group="ur_manipulator">
       <joint name="${prefix}elbow_joint" value="0" />
       <joint name="${prefix}shoulder_lift_joint" value="-1.5707" />
@@ -23,5 +35,5 @@
       <joint name="${prefix}wrist_3_joint" value="0" />
     </group_state>
-    <group_state name="${prefix}up" group="${prefix}${name}_manipulator">
+    <group_state name="${prefix}up" group="ur_manipulator">
       <joint name="${prefix}elbow_joint" value="0" />
       <joint name="${prefix}shoulder_lift_joint" value="-1.5707" />
@@ -31,5 +43,5 @@
       <joint name="${prefix}wrist_3_joint" value="0" />
     </group_state>
-    <group_state name="${prefix}test_configuration" group="${prefix}${name}_manipulator">
+    <group_state name="${prefix}test_configuration" group="ur_manipulator">
       <joint name="${prefix}elbow_joint" value="1.4" />
       <joint name="${prefix}shoulder_lift_joint" value="-1.62" />
@@ -39,6 +51,14 @@
       <joint name="${prefix}wrist_3_joint" value="-0.11" />
     </group_state>
+    <group_state name="gripper_open" group="${prefix}${name}_gripper">
+        <joint name="finger_joint" value="0"/>
+    </group_state>
+    <group_state name="gripper_close" group="${prefix}${name}_gripper">
+        <joint name="finger_joint" value="0.7"/>
+    </group_state>
     <!--END EFFECTOR - Purpose - Represent information about an end effector.-->
+    <end_effector name="robotiq_140_gripper" parent_link="ee_link" group="${prefix}${name}_gripper" parent_group="ur_manipulator"/>
     <!--VIRTUAL JOINT - Purpose - this element defines a virtual joint between a robot link and an external frame of reference (considered fixed with respect to the robot)-->
+    <virtual_joint name="virtual_joint" type="fixed" parent_frame="world" child_link="base_link" />
     <!--DISABLE COLLISIONS - By default it is assumed that any link of the robot could potentially come into collision with any other link in the robot. This tag disables collision checking between a specified pair of links. -->
     <disable_collisions link1="${prefix}base_link" link2="${prefix}base_link_inertia" reason="Adjacent" />
@@ -53,4 +73,54 @@
     <disable_collisions link1="${prefix}wrist_1_link" link2="${prefix}wrist_3_link" reason="Never" />
     <disable_collisions link1="${prefix}wrist_2_link" link2="${prefix}wrist_3_link" reason="Adjacent" />
+    <disable_collisions link1="${prefix}wrist_3_link" link2="robotiq_140_base_link" reason="Adjacent" />
+    <disable_collisions link1="${prefix}tool0" link2="robotiq_140_base_link" reason="Never" />
+    <disable_collisions link1="${prefix}tool0" link2="right_outer_knuckle" reason="Never" />
+    <disable_collisions link1="${prefix}tool0" link2="right_outer_finger" reason="Never" />
+    <disable_collisions link1="${prefix}tool0" link2="right_inner_knuckle" reason="Never" />
+    <disable_collisions link1="${prefix}tool0" link2="right_inner_finger" reason="Never" />
+    <disable_collisions link1="${prefix}tool0" link2="left_outer_knuckle" reason="Never" />
+    <disable_collisions link1="${prefix}tool0" link2="left_outer_finger" reason="Never" />
+    <disable_collisions link1="${prefix}tool0" link2="left_inner_knuckle" reason="Never" />
+    <disable_collisions link1="${prefix}tool0" link2="left_inner_finger" reason="Never" />
+    <disable_collisions link1="${prefix}tool0" link2="right_inner_finger_pad" reason="Never" />
+    <disable_collisions link1="${prefix}tool0" link2="left_inner_finger_pad" reason="Never" />
+    <disable_collisions link1="robotiq_140_base_link" link2="right_outer_knuckle" reason="Adjacent" />
+    <disable_collisions link1="robotiq_140_base_link" link2="right_outer_finger" reason="Never" />
+    <disable_collisions link1="robotiq_140_base_link" link2="right_inner_knuckle" reason="Adjacent" />
+    <disable_collisions link1="robotiq_140_base_link" link2="right_inner_finger" reason="Never" />
+    <disable_collisions link1="robotiq_140_base_link" link2="left_outer_knuckle" reason="Adjacent" />
+    <disable_collisions link1="robotiq_140_base_link" link2="left_outer_finger" reason="Never" />
+    <disable_collisions link1="robotiq_140_base_link" link2="left_inner_knuckle" reason="Adjacent" />
+    <disable_collisions link1="robotiq_140_base_link" link2="left_inner_finger" reason="Never" />
+    <disable_collisions link1="robotiq_140_base_link" link2="right_inner_finger_pad" reason="Never" />
+    <disable_collisions link1="robotiq_140_base_link" link2="left_inner_finger_pad" reason="Never" />
+    <disable_collisions link1="right_outer_knuckle" link2="robotiq_140_base_link" reason="Adjacent" />
+    <disable_collisions link1="right_outer_knuckle" link2="right_outer_finger" reason="Adjacent" />
+    <disable_collisions link1="right_outer_knuckle" link2="right_inner_knuckle" reason="Never" />
+    <disable_collisions link1="right_outer_knuckle" link2="right_inner_finger" reason="Never" />
+    <disable_collisions link1="right_outer_knuckle" link2="left_outer_knuckle" reason="Never" />
+    <disable_collisions link1="right_outer_knuckle" link2="left_outer_finger" reason="Never" />
+    <disable_collisions link1="right_outer_knuckle" link2="left_inner_knuckle" reason="Never" />
+    <disable_collisions link1="right_outer_knuckle" link2="left_inner_finger" reason="Never" />
+    <disable_collisions link1="right_outer_knuckle" link2="right_inner_finger_pad" reason="Never" />
+    <disable_collisions link1="right_outer_knuckle" link2="left_inner_finger_pad" reason="Never" />
+    <disable_collisions link1="left_outer_knuckle" link2="robotiq_140_base_link" reason="Adjacent" />
+    <disable_collisions link1="left_outer_knuckle" link2="right_outer_finger" reason="Never" />
+    <disable_collisions link1="left_outer_knuckle" link2="right_inner_knuckle" reason="Never" />
+    <disable_collisions link1="left_outer_knuckle" link2="right_inner_finger" reason="Never" />
+    <disable_collisions link1="left_outer_knuckle" link2="right_outer_knuckle" reason="Never" />
+    <disable_collisions link1="left_outer_knuckle" link2="left_outer_finger" reason="Adjacent" />
+    <disable_collisions link1="left_outer_knuckle" link2="left_inner_knuckle" reason="Never" />
+    <disable_collisions link1="left_outer_knuckle" link2="left_inner_finger" reason="Never" />
+    <disable_collisions link1="left_outer_knuckle" link2="right_inner_finger_pad" reason="Never" />
+    <disable_collisions link1="left_outer_knuckle" link2="left_inner_finger_pad" reason="Never" />
+    <disable_collisions link1="right_outer_finger" link2="right_outer_knuckle" reason="Adjacent" />
+    <disable_collisions link1="right_outer_finger" link2="right_inner_finger" reason="Adjacent" />
+    <disable_collisions link1="right_inner_finger" link2="right_inner_knuckle" reason="Adjacent" />
+    <disable_collisions link1="right_inner_finger" link2="right_inner_finger_pad" reason="Adjacent" />
+    <disable_collisions link1="left_outer_finger" link2="left_outer_knuckle" reason="Adjacent" />
+    <disable_collisions link1="left_outer_finger" link2="left_inner_finger" reason="Adjacent" />
+    <disable_collisions link1="left_inner_finger" link2="left_inner_knuckle" reason="Adjacent" />
+    <disable_collisions link1="left_inner_finger" link2="left_inner_finger_pad" reason="Adjacent" />
   </xacro:macro>
 </robot>

Commit message: add_gripper

File: ur_moveit_config/srdf/ur_macro.srdf.xacro (robot description, xacro)
@@ -1,5 +1,5 @@
 <?xml version="1.0" encoding="UTF-8"?>
 <robot xmlns:xacro="http://wiki.ros.org/xacro">
-<!--This does not replace URDF, and is not an extension of URDF.
+  <!--This does not replace URDF, and is not an extension of URDF.
     This is a format for representing semantic information about the robot structure.
     A URDF file must exist for this robot as well, where the joints and the links that are referenced are defined
@@ -14,5 +14,5 @@
       <chain base_link="${prefix}base_link" tip_link="${prefix}ee_link" />
     </group>
-    <group name="${prefix}${name}_gripper">
+    <group name="ur_gripper">
       <joint name="finger_joint"/>
       <joint name="left_inner_knuckle_joint" />
@@ -51,12 +51,12 @@
       <joint name="${prefix}wrist_3_joint" value="-0.11" />
     </group_state>
-    <group_state name="gripper_open" group="${prefix}${name}_gripper">
-        <joint name="finger_joint" value="0"/>
+    <group_state name="gripper_open" group="ur_gripper">
+      <joint name="finger_joint" value="0"/>
     </group_state>
-    <group_state name="gripper_close" group="${prefix}${name}_gripper">
-        <joint name="finger_joint" value="0.7"/>
+    <group_state name="gripper_close" group="ur_gripper">
+      <joint name="finger_joint" value="0.699"/>
     </group_state>
     <!--END EFFECTOR - Purpose - Represent information about an end effector.-->
-    <end_effector name="robotiq_140_gripper" parent_link="ee_link" group="${prefix}${name}_gripper" parent_group="ur_manipulator"/>
+    <end_effector name="robotiq_140_gripper" parent_link="ee_link" group="ur_gripper" parent_group="ur_manipulator"/>
     <!--VIRTUAL JOINT - Purpose - this element defines a virtual joint between a robot link and an external frame of reference (considered fixed with respect to the robot)-->
     <virtual_joint name="virtual_joint" type="fixed" parent_frame="world" child_link="base_link" />
